Commit message: Tiago added
Signed-off-by: Francisco Martín Rico <fmrico@gmail.com>

File: kobuki/definition/sim/hokuyo.urdf.xacro (robot description, xacro)
@@ -13,5 +13,5 @@
       <origin xyz="0 0 0" rpy="0 0 0"/>
       <geometry>
-        <mesh filename="package://robots/definition/sim/hokuyo.dae"/>
+        <mesh filename="package://ir_kobuki/definition/sim/hokuyo.dae"/>
       </geometry>
       </visual>

File: kobuki/definition/sim/kobuki_hexagons_asus_xtion_pro.urdf.xacro (robot description, xacro)
@@ -6,20 +6,20 @@
 -->
 <robot name="turtlebot" xmlns:xacro="http://ros.org/wiki/xacro">
-	<xacro:include filename="$(find robots)/definition/sim/urdf/common_properties.urdf.xacro"/>
-  <xacro:include filename="$(find robots)/definition/sim/urdf/turtlebot_properties.urdf.xacro"/>
+	<xacro:include filename="$(find ir_kobuki)/definition/sim/urdf/common_properties.urdf.xacro"/>
+  <xacro:include filename="$(find ir_kobuki)/definition/sim/urdf/turtlebot_properties.urdf.xacro"/>
   <!-- Bases -->
-  <xacro:include filename="$(find robots)/definition/sim/urdf/create.urdf.xacro"/>
-  <xacro:include filename="$(find robots)/definition/sim/urdf/kobuki.urdf.xacro" />
+  <xacro:include filename="$(find ir_kobuki)/definition/sim/urdf/create.urdf.xacro"/>
+  <xacro:include filename="$(find ir_kobuki)/definition/sim/urdf/kobuki.urdf.xacro" />
   <!-- Stacks -->
-  <xacro:include filename="$(find robots)/definition/sim/urdf/stacks/circles.urdf.xacro"/>
-  <xacro:include filename="$(find robots)/definition/sim/urdf/stacks/hexagons.urdf.xacro"/>
+  <xacro:include filename="$(find ir_kobuki)/definition/sim/urdf/stacks/circles.urdf.xacro"/>
+  <xacro:include filename="$(find ir_kobuki)/definition/sim/urdf/stacks/hexagons.urdf.xacro"/>
   <!-- 3D Sensors -->
-  <xacro:include filename="$(find robots)/definition/sim/urdf/sensors/kinect.urdf.xacro"/>
-  <xacro:include filename="$(find robots)/definition/sim/urdf/sensors/asus_xtion_pro.urdf.xacro"/>
-  <xacro:include filename="$(find robots)/definition/sim/urdf/sensors/asus_xtion_pro_offset.urdf.xacro"/>
+  <xacro:include filename="$(find ir_kobuki)/definition/sim/urdf/sensors/kinect.urdf.xacro"/>
+  <xacro:include filename="$(find ir_kobuki)/definition/sim/urdf/sensors/asus_xtion_pro.urdf.xacro"/>
+  <xacro:include filename="$(find ir_kobuki)/definition/sim/urdf/sensors/asus_xtion_pro_offset.urdf.xacro"/>
   <xacro:kobuki/>
   <xacro:stack_hexagons                 parent="base_link"/>
   <xacro:sensor_asus_xtion_pro          parent="base_link"/>
-  <xacro:include filename="$(find robots)/definition/sim/hokuyo.urdf.xacro" />
+  <xacro:include filename="$(find ir_kobuki)/definition/sim/hokuyo.urdf.xacro" />
   <xacro:hokuyo name="laser0" parent="base_link" ros_topic="scan" update_rate="40" ray_count="1081" min_angle="135" max_angle="-135">
       <origin xyz="0.0 0.0 0.08" rpy="${M_PI} 0 0"/>

File: kobuki/definition/sim/urdf/create.urdf.xacro (robot description, xacro)
@@ -2,5 +2,5 @@
 <robot name="turtlebot_hardware" xmlns:xacro="http://ros.org/wiki/xacro">
   <!-- Macro for TurtleBot body. Including Gazebo extensions, but does not include Kinect -->
-  <xacro:include filename="$(find robots)/definition/sim/urdf/create_gazebo.urdf.xacro"/>
+  <xacro:include filename="$(find ir_kobuki)/definition/sim/urdf/create_gazebo.urdf.xacro"/>
   <xacro:property name="base_x" value="0.33" />
   <xacro:property name="base_y" value="0.33" />

File: kobuki/definition/sim/urdf/kobuki.urdf.xacro (robot description, xacro)
@@ -7,6 +7,6 @@
  -->
 <robot name="kobuki" xmlns:xacro="http://ros.org/wiki/xacro">
-  <xacro:include filename="$(find robots)/definition/sim/urdf/common_properties.urdf.xacro"/>
-  <xacro:include filename="$(find robots)/definition/sim/urdf/kobuki_gazebo.urdf.xacro"/>
+  <xacro:include filename="$(find ir_kobuki)/definition/sim/urdf/common_properties.urdf.xacro"/>
+  <xacro:include filename="$(find ir_kobuki)/definition/sim/urdf/kobuki_gazebo.urdf.xacro"/>
   <!-- Kobuki -->
   <xacro:macro name="kobuki">
@@ -30,5 +30,5 @@
         <geometry>
           <!-- new mesh -->
-          <mesh filename="package://robots/definition/sim/meshes/main_body.dae" />
+          <mesh filename="package://ir_kobuki/definition/sim/meshes/main_body.dae" />
         </geometry>
         <origin xyz="0.001 0 0.05199" rpy="0 0 0"/>
@@ -65,5 +65,5 @@
       <visual>
         <geometry>
-          <mesh filename="package://robots/definition/sim/meshes/wheel.dae"/>
+          <mesh filename="package://ir_kobuki/definition/sim/meshes/wheel.dae"/>
         </geometry>
         <origin xyz="0 0 0" rpy="0 0 0"/>
@@ -92,5 +92,5 @@
       <visual>
         <geometry>
-          <mesh filename="package://robots/definition/sim/meshes/wheel.dae"/>
+          <mesh filename="package://ir_kobuki/definition/sim/meshes/wheel.dae"/>
         </geometry>
         <origin xyz="0 0 0" rpy="0 0 0"/>

File: kobuki/definition/sim/urdf/sensors/astra.urdf.xacro (robot description, xacro)
@@ -1,6 +1,6 @@
 <?xml version="1.0"?>
 <robot name="sensor_astra" xmlns:xacro="http://ros.org/wiki/xacro">
-  <xacro:include filename="$(find robots)/definition/sim/urdf/turtlebot_gazebo.urdf.xacro"/>
-  <xacro:include filename="$(find robots)/definition/sim/urdf/turtlebot_properties.urdf.xacro"/>
+  <xacro:include filename="$(find ir_kobuki)/definition/sim/urdf/turtlebot_gazebo.urdf.xacro"/>
+  <xacro:include filename="$(find ir_kobuki)/definition/sim/urdf/turtlebot_properties.urdf.xacro"/>
   <!-- Xacro properties -->
   <xacro:property name="astra_cam_py" value="-0.0125"/>
@@ -33,5 +33,5 @@
         <origin xyz="-0.04 0.02 -0.01" rpy="${M_PI/2} 0 ${M_PI/2}"/>
         <geometry>
-          <mesh filename="package://robots/definition/sim/meshes/sensors/astra.dae" scale="${astra_dae_display_scale} ${astra_dae_display_scale} ${astra_dae_display_scale}"/>
+          <mesh filename="package://ir_kobuki/definition/sim/meshes/sensors/astra.dae" scale="${astra_dae_display_scale} ${astra_dae_display_scale} ${astra_dae_display_scale}"/>
         </geometry>
       </visual>

File: kobuki/definition/sim/urdf/sensors/asus_xtion_pro.urdf.xacro (robot description, xacro)
@@ -1,6 +1,6 @@
 <?xml version="1.0"?>
 <robot name="sensor_asus_xtion_pro" xmlns:xacro="http://ros.org/wiki/xacro">
-  <xacro:include filename="$(find robots)/definition/sim/urdf/turtlebot_gazebo.urdf.xacro"/>
-  <xacro:include filename="$(find robots)/definition/sim/urdf/turtlebot_properties.urdf.xacro"/>
+  <xacro:include filename="$(find ir_kobuki)/definition/sim/urdf/turtlebot_gazebo.urdf.xacro"/>
+  <xacro:include filename="$(find ir_kobuki)/definition/sim/urdf/turtlebot_properties.urdf.xacro"/>
   <!-- Xacro properties -->
   <xacro:property name="M_SCALE" value="0.001"/>
@@ -33,5 +33,5 @@
         <origin xyz="-0.015 0.0035 0.004" rpy="0 0 0"/>
         <geometry>
-          <mesh filename="package://robots/definition/sim/meshes/sensors/xtion_pro_camera.dae"/>
+          <mesh filename="package://ir_kobuki/definition/sim/meshes/sensors/xtion_pro_camera.dae"/>
         </geometry>
       </visual>
@@ -74,5 +74,5 @@
         <origin xyz="0 0 0" rpy="${-M_PI/2} 0 0"/>
         <geometry>
-          <mesh filename="package://robots/definition/sim/meshes/sensors/xtion_pro_stack.dae"/>
+          <mesh filename="package://ir_kobuki/definition/sim/meshes/sensors/xtion_pro_stack.dae"/>
         </geometry>
       </visual>

File: kobuki/definition/sim/urdf/sensors/asus_xtion_pro_offset.urdf.xacro (robot description, xacro)
@@ -1,6 +1,6 @@
 <?xml version="1.0"?>
 <robot name="sensor_asus_xtion_pro_offset" xmlns:xacro="http://ros.org/wiki/xacro">
-  <xacro:include filename="$(find robots)/definition/sim/urdf/turtlebot_gazebo.urdf.xacro"/>
-  <xacro:include filename="$(find robots)/definition/sim/urdf/turtlebot_properties.urdf.xacro"/>
+  <xacro:include filename="$(find ir_kobuki)/definition/sim/urdf/turtlebot_gazebo.urdf.xacro"/>
+  <xacro:include filename="$(find ir_kobuki)/definition/sim/urdf/turtlebot_properties.urdf.xacro"/>
   <!-- Xacro properties -->
   <xacro:property name="M_SCALE" value="0.001"/>
@@ -33,5 +33,5 @@
         <origin xyz="-0.01 0 0" rpy="${-M_PI/2} -${M_PI} ${-M_PI/2}"/>
         <geometry>
-          <mesh filename="package://robots/definition/sim/meshes/sensors/asus_xtion_pro_live.dae" scale="${M_SCALE} ${M_SCALE} ${M_SCALE}"/>
+          <mesh filename="package://ir_kobuki/definition/sim/meshes/sensors/asus_xtion_pro_live.dae" scale="${M_SCALE} ${M_SCALE} ${M_SCALE}"/>
         </geometry>
       </visual>

File: kobuki/definition/sim/urdf/sensors/kinect.urdf.xacro (robot description, xacro)
@@ -1,6 +1,6 @@
 <?xml version="1.0"?>
 <robot name="sensor_kinect" xmlns:xacro="http://ros.org/wiki/xacro">
-  <xacro:include filename="$(find robots)/definition/sim/urdf/turtlebot_gazebo.urdf.xacro"/>
-  <xacro:include filename="$(find robots)/definition/sim/urdf/turtlebot_properties.urdf.xacro"/>
+  <xacro:include filename="$(find ir_kobuki)/definition/sim/urdf/turtlebot_gazebo.urdf.xacro"/>
+  <xacro:include filename="$(find ir_kobuki)/definition/sim/urdf/turtlebot_properties.urdf.xacro"/>
   <xacro:property name="kinect_cam_py" value="-0.0125"/>
   <!-- Parameterised in part by the values in turtlebot_properties.urdf.xacro -->
@@ -27,5 +27,5 @@
        <origin xyz="0 0 0" rpy="0 0 ${M_PI/2}"/>
         <geometry>
-         <mesh filename="package://robots/definition/sim/meshes/sensors/kinect.dae"/>
+         <mesh filename="package://ir_kobuki/definition/sim/meshes/sensors/kinect.dae"/>
         </geometry>
       </visual>

File: kobuki/definition/sim/urdf/sensors/r200.urdf.xacro (robot description, xacro)
@@ -1,6 +1,6 @@
 <?xml version="1.0"?>
 <robot name="sensor_r200" xmlns:xacro="http://ros.org/wiki/xacro">
-  <xacro:include filename="$(find robots)/definition/sim/urdf/turtlebot_gazebo.urdf.xacro"/>
-  <xacro:include filename="$(find robots)/definition/sim/urdf/turtlebot_properties.urdf.xacro"/>
+  <xacro:include filename="$(find ir_kobuki)/definition/sim/urdf/turtlebot_gazebo.urdf.xacro"/>
+  <xacro:include filename="$(find ir_kobuki)/definition/sim/urdf/turtlebot_properties.urdf.xacro"/>
   <!-- Mount and camera parameters -->
   <xacro:property name="pole_px" value="-0.103" />
@@ -35,5 +35,5 @@
        <origin xyz="${-r200_bracket_end_width/2} ${r200_bracket_end_offset_py} ${r200_bracket_end_offset_pz}" rpy="0 0 ${-M_PI/2}"/>
         <geometry>
-         <mesh filename="package://robots/definition/sim/meshes/sensors/r200_bracket_end.stl" scale="0.001 0.001 0.001"/>
+         <mesh filename="package://ir_kobuki/definition/sim/meshes/sensors/r200_bracket_end.stl" scale="0.001 0.001 0.001"/>
         </geometry>
         <xacro:insert_block name="material_dark_grey" />
@@ -50,5 +50,5 @@
        <origin xyz="0 0 0" rpy="0 0 ${M_PI/2}"/>
         <geometry>
-         <mesh filename="package://robots/definition/sim/meshes/sensors/r200_bracket.stl" scale="0.001 0.001 0.001"/>
+         <mesh filename="package://ir_kobuki/definition/sim/meshes/sensors/r200_bracket.stl" scale="0.001 0.001 0.001"/>
         </geometry>
         <xacro:insert_block name="material_dark_grey" />
@@ -65,5 +65,5 @@
        <origin xyz="${r200_bracket_end_width/2} 0 ${-r200_bracket_end_offset_pz}" rpy="0 0 ${M_PI/2}"/>
         <geometry>
-         <mesh filename="package://robots/definition/sim/meshes/sensors/r200_bracket_end.stl" scale="0.001 0.001 0.001"/>
+         <mesh filename="package://ir_kobuki/definition/sim/meshes/sensors/r200_bracket_end.stl" scale="0.001 0.001 0.001"/>
         </geometry>
         <xacro:insert_block name="material_dark_grey" />
@@ -80,5 +80,5 @@
        <origin xyz="0 0 0" rpy="${M_PI/2} 0 ${M_PI/2}"/>
         <geometry>
-         <mesh filename="package://robots/definition/sim/meshes/sensors/r200.dae" />
+         <mesh filename="package://ir_kobuki/definition/sim/meshes/sensors/r200.dae" />
         </geometry>
       </visual>

File: kobuki/definition/sim/urdf/stacks/circles.urdf.xacro (robot description, xacro)
@@ -18,5 +18,5 @@
         <origin xyz=" 0 0 0 " rpy="0 0 0" />
         <geometry>
-          <mesh filename="package://robots/definition/sim/meshes/stacks/circles/68-02403-125_Spacer.dae"/>
+          <mesh filename="package://ir_kobuki/definition/sim/meshes/stacks/circles/68-02403-125_Spacer.dae"/>
         </geometry>
       </visual>
@@ -46,5 +46,5 @@
         <origin xyz=" 0 0 0 " rpy="0 0 0" />
         <geometry>
-          <mesh filename="package://robots/definition/sim/meshes/stacks/circles/68-04552-1000-RA_Turtlebot_M-F_Standoff.dae"/>
+          <mesh filename="package://ir_kobuki/definition/sim/meshes/stacks/circles/68-04552-1000-RA_Turtlebot_M-F_Standoff.dae"/>
         </geometry>
       </visual>
@@ -74,5 +74,5 @@
         <origin xyz=" 0 0 0 " rpy="0 0 0" />
         <geometry>
-          <mesh filename="package://robots/definition/sim/meshes/stacks/circles/68-04552-2000-RA_Turtlebot_M-F_Standoff.dae"/>
+          <mesh filename="package://ir_kobuki/definition/sim/meshes/stacks/circles/68-04552-2000-RA_Turtlebot_M-F_Standoff.dae"/>
         </geometry>
       </visual>
@@ -102,5 +102,5 @@
         <origin xyz=" 0 0 0 " rpy="0 0 0" />
         <geometry>
-          <mesh filename="package://robots/definition/sim/meshes/stacks/circles/68-02421-8000-RA_Turtlebot_F-F_Standoff.dae"/>
+          <mesh filename="package://ir_kobuki/definition/sim/meshes/stacks/circles/68-02421-8000-RA_Turtlebot_F-F_Standoff.dae"/>
         </geometry>
       </visual>
@@ -130,5 +130,5 @@
         <origin xyz=" 0 0 0 " rpy="0 0 0" />
         <geometry>
-          <mesh filename="package://robots/definition/sim/meshes/stacks/circles/68-04556-RA_Kinect_Standoff_Assy.dae"/>
+          <mesh filename="package://ir_kobuki/definition/sim/meshes/stacks/circles/68-04556-RA_Kinect_Standoff_Assy.dae"/>
         </geometry>
       </visual>
@@ -162,5 +162,5 @@
         <origin xyz=" 0 0 0 " rpy="0 0 0" />
         <geometry>
-          <mesh filename="package://robots/definition/sim/meshes/stacks/circles/plate_0_logo.dae"/>
+          <mesh filename="package://ir_kobuki/definition/sim/meshes/stacks/circles/plate_0_logo.dae"/>
         </geometry>
       </visual>
@@ -192,5 +192,5 @@
         <origin xyz=" 0 0 0 " rpy="0 0 0" />
         <geometry>
-          <mesh filename="package://robots/definition/sim/meshes/stacks/circles/plate_1_logo.dae"/>
+          <mesh filename="package://ir_kobuki/definition/sim/meshes/stacks/circles/plate_1_logo.dae"/>
         </geometry>
       </visual>
@@ -222,5 +222,5 @@
         <origin xyz=" 0 0 0 " rpy="0 0 0" />
         <geometry>
-          <mesh filename="package://robots/definition/sim/meshes/stacks/circles/plate_1_logo.dae"/>
+          <mesh filename="package://ir_kobuki/definition/sim/meshes/stacks/circles/plate_1_logo.dae"/>
         </geometry>
       </visual>
@@ -254,5 +254,5 @@
         <origin xyz=" 0 0 0 " rpy="0 0 0" />
         <geometry>
-          <mesh filename="package://robots/definition/sim/meshes/stacks/circles/plate_2_logo.dae"/>
+          <mesh filename="package://ir_kobuki/definition/sim/meshes/stacks/circles/plate_2_logo.dae"/>
         </geometry>
       </visual>

File: kobuki/definition/sim/urdf/stacks/hexagons.urdf.xacro (robot description, xacro)
@@ -4,5 +4,5 @@
  -->
 <robot name="stack_hexagons" xmlns:xacro="http://ros.org/wiki/xacro">
-  <xacro:include filename="$(find robots)/definition/sim/urdf/common_properties.urdf.xacro"/>
+  <xacro:include filename="$(find ir_kobuki)/definition/sim/urdf/common_properties.urdf.xacro"/>
   <!-- Xacro properties -->
   <xacro:property name="M_SCALE" value="0.001"/>
@@ -19,5 +19,5 @@
         <origin xyz="0 0 0" rpy="0 0 0"/>
         <geometry>
-          <mesh filename="package://robots/definition/sim/meshes/stacks/hexagons/pole_bottom.dae"/>
+          <mesh filename="package://ir_kobuki/definition/sim/meshes/stacks/hexagons/pole_bottom.dae"/>
         </geometry>
       </visual>
@@ -47,5 +47,5 @@
         <origin xyz="0 0 0" rpy="0 ${M_PI} 0"/>
         <geometry>
-          <mesh filename="package://robots/definition/sim/meshes/stacks/hexagons/pole_middle.dae"/>
+          <mesh filename="package://ir_kobuki/definition/sim/meshes/stacks/hexagons/pole_middle.dae"/>
         </geometry>
       </visual>
@@ -75,5 +75,5 @@
         <origin xyz=" 0 0 0" rpy="0 0 0"/>
         <geometry>
-          <mesh filename="package://robots/definition/sim/meshes/stacks/hexagons/pole_top.dae"/>
+          <mesh filename="package://ir_kobuki/definition/sim/meshes/stacks/hexagons/pole_top.dae"/>
         </geometry>
       </visual>
@@ -103,5 +103,5 @@
         <origin xyz="0 0 -0.01" rpy="0 0 0"/>
         <geometry>
-          <mesh filename="package://robots/definition/sim/meshes/sensors/sensor_pole.dae" />
+          <mesh filename="package://ir_kobuki/definition/sim/meshes/sensors/sensor_pole.dae" />
         </geometry>
       </visual>
@@ -142,5 +142,5 @@
         <origin xyz="0 0 0" rpy="0 0 0"/>
         <geometry>
-          <mesh filename="package://robots/definition/sim/meshes/stacks/hexagons/plate_bottom.dae"/>
+          <mesh filename="package://ir_kobuki/definition/sim/meshes/stacks/hexagons/plate_bottom.dae"/>
         </geometry>
       </visual>
@@ -172,5 +172,5 @@
         <origin xyz="0 0 0" rpy="0 0 0"/>
         <geometry>
-          <mesh filename="package://robots/definition/sim/meshes/stacks/hexagons/plate_middle.dae"/>
+          <mesh filename="package://ir_kobuki/definition/sim/meshes/stacks/hexagons/plate_middle.dae"/>
         </geometry>
       </visual>
@@ -204,5 +204,5 @@
         <origin xyz="0 0 0" rpy="0 0 0"/>
         <geometry>
-          <mesh filename="package://robots/definition/sim/meshes/stacks/hexagons/plate_top.dae"/>
+          <mesh filename="package://ir_kobuki/definition/sim/meshes/stacks/hexagons/plate_top.dae"/>
         </geometry>
       </visual>

File: kobuki/definition/sim/urdf/turtlebot_common_library.urdf.xacro (robot description, xacro)
@@ -5,5 +5,5 @@
 <robot xmlns:xacro="http://ros.org/wiki/xacro">
   <!-- General -->
-  <xacro:include filename="$(find robots)/definition/sim/urdf/common_properties.urdf.xacro"/>
-  <xacro:include filename="$(find robots)/definition/sim/urdf/turtlebot_properties.urdf.xacro"/>
+  <xacro:include filename="$(find ir_kobuki)/definition/sim/urdf/common_properties.urdf.xacro"/>
+  <xacro:include filename="$(find ir_kobuki)/definition/sim/urdf/turtlebot_properties.urdf.xacro"/>
 </robot>
